File: Potential Schematics/Registers for PCB/Register/Register.kicad_pcb (KiCad board)
At the start: 2 copper layers, 89.5 x 43.8 mm, 15 parts, among them J1 Conn_01x04_Female, J2 Conn_01x08_Female, U1 74LS02, U10 74LS08, U2 74LS02, U3 74LS02, U4 74LS02, U5 74LS04, U6 74LS04, U7 74LS08, U8 74LS08, U9 74LS08

Commit message: Finished PCB designes for Multiplexer and Registers
Parts:
-  : renamed from G***; value LOGO -> (none)
Changed lines of the file:
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@@
   (module Graphics:Real_Logo (layer F.Cu)
     (at 141.605 90.17 180)
-    (fp_text reference G*** (at 0 0 180) (layer F.SilkS) hide
+    (fp_text reference " " (at 4.445 -7.62 180) (layer F.SilkS) hide
       (effects (font (size 1.524 1.524) (thickness 0.3)))
     )
-    (fp_text value LOGO (at 0.75 0 180) (layer F.SilkS) hide
+    (fp_text value " " (at 0.75 -6.985 180) (layer F.SilkS) hide
       (effects (font (size 1.524 1.524) (thickness 0.3)))
     )
