File: Potential Schematics/Registers for PCB/Multiplexer/PowerFor08s.sch (KiCad schematic (older format))
At the start: 66 parts, among them U14 74LS08, U15 74LS08, U16 74LS08, U17 74LS08, U18 74LS08, U19 74LS08, U2 74LS08, U20 74LS08, U21 74LS08, U22 74LS08, U23 74LS08, U24 74LS08, U26 74LS08, U27 74LS08, U28 74LS08, U29 74LS08, U3 74LS08, U30 74LS08, U31 74LS08, U32 74LS08, U33 74LS08, U38 74LS08, U39 74LS08, U4 74LS08, U40 74LS08, U41 74LS08, U42 74LS08, U43 74LS08, U44 74LS08, U45 74LS08, U47 74LS08, U48 74LS08, U49 74LS08, U5 74LS08, U50 74LS08, U51 74LS08, U52 74LS08, U53 74LS08, U54 74LS08, U59 74LS08, U6 74LS08, U60 74LS08, U61 74LS08, U62 74LS08, U63 74LS08, U64 74LS08, U65 74LS08, U66 74LS08, U68 74LS08, U69 74LS08, U7 74LS08, U70 74LS08, U71 74LS08, U72 74LS08, U73 74LS08, U74 74LS08, U75 74LS08, U8 74LS08, U80 74LS08, U81 74LS08, U82 74LS08, U83 74LS08, U84 74LS08, U85 74LS08, U86 74LS08, U9 74LS08

Commit message: Updated PCB and is ready to be ordered
Parts:
- added U87: 74LS08, symbol 74xx:74LS08
Changed lines of the file:
@@
 L power:VCC #PWR?
 U 1 1 5BC2D82C
-P 5200 700
+P 6700 650
 AR Path="/5BC2C594/5BC2D82C" Ref="#PWR?"  Part="1"
 AR Path="/5BC2D2C8/5BC2D82C" Ref="#PWR0147"  Part="1"
-F 0 "#PWR0147" H 5200 550 50  0001 C CNN
-F 1 "VCC" H 5217 873 50  0000 C CNN
-F 2 "" H 5200 700 50  0001 C CNN
-F 3 "" H 5200 700 50  0001 C CNN
-	1    5200 700
+F 0 "#PWR0147" H 6700 500 50  0001 C CNN
+F 1 "VCC" H 6717 823 50  0000 C CNN
+F 2 "" H 6700 650 50  0001 C CNN
+F 3 "" H 6700 650 50  0001 C CNN
+	1    6700 650
 	1    0    0    -1
 $EndComp
@@
 L power:VCC #PWR?
 U 1 1 5BC2D83F
-P 5950 700
+P 7450 650
 AR Path="/5BC2C594/5BC2D83F" Ref="#PWR?"  Part="1"
 AR Path="/5BC2D2C8/5BC2D83F" Ref="#PWR0149"  Part="1"
-F 0 "#PWR0149" H 5950 550 50  0001 C CNN
-F 1 "VCC" H 5967 873 50  0000 C CNN
-F 2 "" H 5950 700 50  0001 C CNN
-F 3 "" H 5950 700 50  0001 C CNN
-	1    5950 700
+F 0 "#PWR0149" H 7450 500 50  0001 C CNN
+F 1 "VCC" H 7467 823 50  0000 C CNN
+F 2 "" H 7450 650 50  0001 C CNN
+F 3 "" H 7450 650 50  0001 C CNN
+	1    7450 650
 	1    0    0    -1
 $EndComp
@@
 	1    0    0    -1
 $EndComp
+$Comp
+L power:VCC #PWR?
+U 1 1 5BDC7853
+P 5200 700
+AR Path="/5BC2C594/5BDC7853" Ref="#PWR?"  Part="1"
+AR Path="/5BC2D2C8/5BDC7853" Ref="#PWR0269"  Part="1"
+F 0 "#PWR0269" H 5200 550 50  0001 C CNN
+F 1 "VCC" H 5217 873 50  0000 C CNN
+F 2 "" H 5200 700 50  0001 C CNN
+F 3 "" H 5200 700 50  0001 C CNN
+	1    5200 700
+	1    0    0    -1
+$EndComp
+$Comp
+L power:VCC #PWR?
+U 1 1 5BDC7859
+P 5950 700
+AR Path="/5BC2C594/5BDC7859" Ref="#PWR?"  Part="1"
+AR Path="/5BC2D2C8/5BDC7859" Ref="#PWR0270"  Part="1"
+F 0 "#PWR0270" H 5950 550 50  0001 C CNN
+F 1 "VCC" H 5967 873 50  0000 C CNN
+F 2 "" H 5950 700 50  0001 C CNN
+F 3 "" H 5950 700 50  0001 C CNN
+	1    5950 700
+	1    0    0    -1
+$EndComp
+$Comp
+L power:VCC #PWR?
+U 1 1 5BDC78A1
+P 8200 650
+AR Path="/5BC2C594/5BDC78A1" Ref="#PWR?"  Part="1"
+AR Path="/5BC2D2C8/5BDC78A1" Ref="#PWR0271"  Part="1"
+F 0 "#PWR0271" H 8200 500 50  0001 C CNN
+F 1 "VCC" H 8217 823 50  0000 C CNN
+F 2 "" H 8200 650 50  0001 C CNN
+F 3 "" H 8200 650 50  0001 C CNN
+	1    8200 650
+	1    0    0    -1
+$EndComp
+$Comp
+L power:VCC #PWR?
+U 1 1 5BDC78A7
+P 8950 650
+AR Path="/5BC2C594/5BDC78A7" Ref="#PWR?"  Part="1"
+AR Path="/5BC2D2C8/5BDC78A7" Ref="#PWR0272"  Part="1"
+F 0 "#PWR0272" H 8950 500 50  0001 C CNN
+F 1 "VCC" H 8967 823 50  0000 C CNN
+F 2 "" H 8950 650 50  0001 C CNN
+F 3 "" H 8950 650 50  0001 C CNN
+	1    8950 650
+	1    0    0    -1
+$EndComp
+$Comp
+L power:VCC #PWR?
+U 1 1 5BDC85D3
+P 9700 650
+AR Path="/5BC2C594/5BDC85D3" Ref="#PWR?"  Part="1"
+AR Path="/5BC2D2C8/5BDC85D3" Ref="#PWR0273"  Part="1"
+F 0 "#PWR0273" H 9700 500 50  0001 C CNN
+F 1 "VCC" H 9717 823 50  0000 C CNN
+F 2 "" H 9700 650 50  0001 C CNN
+F 3 "" H 9700 650 50  0001 C CNN
+	1    9700 650
+	1    0    0    -1
+$EndComp
+$Comp
+L power:VCC #PWR?
+U 1 1 5BDC85D9
+P 10450 650
+AR Path="/5BC2C594/5BDC85D9" Ref="#PWR?"  Part="1"
+AR Path="/5BC2D2C8/5BDC85D9" Ref="#PWR0274"  Part="1"
+F 0 "#PWR0274" H 10450 500 50  0001 C CNN
+F 1 "VCC" H 10467 823 50  0000 C CNN
+F 2 "" H 10450 650 50  0001 C CNN
+F 3 "" H 10450 650 50  0001 C CNN
+	1    10450 650
+	1    0    0    -1
+$EndComp
+$Comp
+L power:VCC #PWR?
+U 1 1 5BDCA8DF
+P 8500 6300
+AR Path="/5BC2C594/5BDCA8DF" Ref="#PWR?"  Part="1"
+AR Path="/5BC2D2C8/5BDCA8DF" Ref="#PWR01"  Part="1"
+F 0 "#PWR01" H 8500 6150 50  0001 C CNN
+F 1 "VCC" H 8517 6473 50  0000 C CNN
+F 2 "" H 8500 6300 50  0001 C CNN
+F 3 "" H 8500 6300 50  0001 C CNN
+	1    8500 6300
+	1    0    0    -1
+$EndComp
+$Comp
+L power:GND #PWR?
+U 1 1 5BDCA8E5
+P 8500 7300
+AR Path="/5BC2C594/5BDCA8E5" Ref="#PWR?"  Part="1"
+AR Path="/5BC2D2C8/5BDCA8E5" Ref="#PWR02"  Part="1"
+F 0 "#PWR02" H 8500 7050 50  0001 C CNN
+F 1 "GND" H 8505 7127 50  0000 C CNN
+F 2 "" H 8500 7300 50  0001 C CNN
+F 3 "" H 8500 7300 50  0001 C CNN
+	1    8500 7300
+	1    0    0    -1
+$EndComp
+$Comp
+L 74xx:74LS08 U87
+U 5 1 5BDCA8EB
+P 8500 6800
+F 0 "U87" H 8730 6846 50  0000 L CNN
+F 1 "74LS08" H 8730 6755 50  0000 L CNN
+F 2 "" H 8500 6800 50  0001 C CNN
+F 3 "http://www.ti.com/lit/gpn/sn74LS08" H 8500 6800 50  0001 C CNN
+	5    8500 6800
+	1    0    0    -1
+$EndComp
