File: Potential Schematics/1-2_Multiplexer.sch (KiCad schematic (older format))
At the start: 4 parts

Commit message: Made Full ALU
Parts:
- gave numbers to parts that had none: 4
Connections:
- net D0: now also U2.4; no longer U2.1
- net D1: now also U5.9; no longer U5.1
- net Out: now also U3.6; no longer U3.3
- net Select: now also U1.3, U5.10; no longer U1.1, U5.2
- new net: U2.6, U3.4
- new net: U3.5, U5.8
- new net: U1.4, U2.5
Changed lines of the file:
@@
 $Descr A4 11693 8268
 encoding utf-8
-Sheet 4 6
-Title ""
+Sheet 13 22
+Title "1:2 Multiplexer"
 Date ""
 Rev "1"
@@
 Out
 $Comp
-L 74LS32 U?
-U 1 1 5B98DCD8
+L 74LS32 U3
+U 2 1 5B98DCD8
 P 7100 3750
-F 0 "U?" H 7100 3800 50  0000 C CNN
+AR Path="/5B990C59/5B990C5E/5B98DA2C/5B98DCD8" Ref="U3"  Part="2"
+AR Path="/5B990C59/5B99BC00/5B98DA2C/5B98DCD8" Ref="U11"  Part="2"
+AR Path="/5B990C59/5B99C896/5B98DA2C/5B98DCD8" Ref="U19"  Part="2"
+AR Path="/5B990C59/5B99C8B8/5B98DA2C/5B98DCD8" Ref="U26"  Part="2"
+F 0 "U19" H 7100 3800 50  0000 C CNN
 F 1 "74LS32" H 7100 3700 50  0000 C CNN
 F 2 "" H 7100 3750 50  0001 C CNN
 F 3 "" H 7100 3750 50  0001 C CNN
-	1    7100 3750
+	2    7100 3750
 	1    0    0    -1
 $EndComp
 $Comp
-L 74LS08 U?
-U 1 1 5B98DCDF
+L 74LS08 U2
+U 2 1 5B98DCDF
 P 5750 3350
-F 0 "U?" H 5750 3400 50  0000 C CNN
+AR Path="/5B990C59/5B990C5E/5B98DA2C/5B98DCDF" Ref="U2"  Part="4"
+AR Path="/5B990C59/5B99BC00/5B98DA2C/5B98DCDF" Ref="U13"  Part="1"
+AR Path="/5B990C59/5B99C896/5B98DA2C/5B98DCDF" Ref="U21"  Part="2"
+AR Path="/5B990C59/5B99C8B8/5B98DA2C/5B98DCDF" Ref="U28"  Part="3"
+F 0 "U21" H 5750 3400 50  0000 C CNN
 F 1 "74LS08" H 5750 3300 50  0000 C CNN
 F 2 "" H 5750 3350 50  0001 C CNN
 F 3 "" H 5750 3350 50  0001 C CNN
-	1    5750 3350
+	2    5750 3350
 	1    0    0    -1
 $EndComp
 $Comp
-L 74LS08 U?
-U 1 1 5B98DCE6
+L 74LS08 U5
+U 3 1 5B98DCE6
 P 5750 4150
-F 0 "U?" H 5750 4200 50  0000 C CNN
+AR Path="/5B990C59/5B990C5E/5B98DA2C/5B98DCE6" Ref="U5"  Part="1"
+AR Path="/5B990C59/5B99BC00/5B98DA2C/5B98DCE6" Ref="U13"  Part="2"
+AR Path="/5B990C59/5B99C896/5B98DA2C/5B98DCE6" Ref="U21"  Part="3"
+AR Path="/5B990C59/5B99C8B8/5B98DA2C/5B98DCE6" Ref="U28"  Part="4"
+F 0 "U21" H 5750 4200 50  0000 C CNN
 F 1 "74LS08" H 5750 4100 50  0000 C CNN
 F 2 "" H 5750 4150 50  0001 C CNN
 F 3 "" H 5750 4150 50  0001 C CNN
-	1    5750 4150
+	3    5750 4150
 	1    0    0    -1
 $EndComp
@@
 	6500 3350 6350 3350
 $Comp
-L 74LS04 U?
-U 1 1 5B98DCF1
+L 74LS04 U1
+U 2 1 5B98DCF1
 P 4750 2700
-F 0 "U?" H 4945 2815 50  0000 C CNN
+AR Path="/5B990C59/5B990C5E/5B98DA2C/5B98DCF1" Ref="U1"  Part="2"
+AR Path="/5B990C59/5B99BC00/5B98DA2C/5B98DCF1" Ref="U10"  Part="2"
+AR Path="/5B990C59/5B99C896/5B98DA2C/5B98DCF1" Ref="U18"  Part="2"
+AR Path="/5B990C59/5B99C8B8/5B98DA2C/5B98DCF1" Ref="U25"  Part="2"
+F 0 "U18" H 4945 2815 50  0000 C CNN
 F 1 "74LS04" H 4940 2575 50  0000 C CNN
 F 2 "" H 4750 2700 50  0001 C CNN
 F 3 "" H 4750 2700 50  0001 C CNN
-	1    4750 2700
+	2    4750 2700
 	0    1    1    0
 $EndComp

Commit message: Adding Multiply Devide
Parts:
- U1: symbol 74LS04 -> 4-bit_processor-rescue:74LS04
- U2, U5: symbol 74LS08 -> 4-bit_processor-rescue:74LS08
- U3: symbol 74LS32 -> 4-bit_processor-rescue:74LS32
Changed lines of the file:
@@
-EESchema Schematic File Version 2
-LIBS:power
-LIBS:device
-LIBS:switches
-LIBS:relays
-LIBS:motors
-LIBS:transistors
-LIBS:conn
-LIBS:linear
-LIBS:regul
-LIBS:74xx
-LIBS:cmos4000
-LIBS:adc-dac
-LIBS:memory
-LIBS:xilinx
-LIBS:microcontrollers
-LIBS:dsp
-LIBS:microchip
-LIBS:analog_switches
-LIBS:motorola
-LIBS:texas
-LIBS:intel
-LIBS:audio
-LIBS:interface
-LIBS:digital-audio
-LIBS:philips
-LIBS:display
-LIBS:cypress
-LIBS:siliconi
-LIBS:opto
-LIBS:atmel
-LIBS:contrib
-LIBS:valves
+EESchema Schematic File Version 4
 LIBS:4-bit_processor-cache
-EELAYER 25 0
+EELAYER 26 0
 EELAYER END
 $Descr A4 11693 8268
 encoding utf-8
-Sheet 13 449
+Sheet 6 451
 Title "1:2 Multiplexer"
 Date "2018-09-14"
@@
 Out
 $Comp
-L 74LS32 U3
+L 4-bit_processor-rescue:74LS32 U3
 U 2 1 5B98DCD8
 P 7100 3750
@@
 $EndComp
 $Comp
-L 74LS08 U2
+L 4-bit_processor-rescue:74LS08 U2
 U 2 1 5B98DCDF
 P 5750 3350
@@
 $EndComp
 $Comp
-L 74LS08 U5
+L 4-bit_processor-rescue:74LS08 U5
 U 3 1 5B98DCE6
 P 5750 4150
@@
 	6500 3350 6350 3350
 $Comp
-L 74LS04 U1
+L 4-bit_processor-rescue:74LS04 U1
 U 2 1 5B98DCF1
 P 4750 2700
@@
 	3250 4050 5150 4050
 Wire Wire Line
-	4400 2250 4750 2250
+	4400 2250 4550 2250
 Wire Wire Line
 	4550 2250 4550 2100
@@
 	4400 4250 4400 2250
 Connection ~ 4550 2250
+Wire Wire Line
+	4550 2250 4750 2250
 $EndSCHEMATC

Commit message: Finished PCB
Parts:
- U2: renamed from U1; footprint (none) -> Daniel_Kopp:DIP-14_300_ELL
- U3, U5: footprint (none) -> Daniel_Kopp:DIP-14_300_ELL
- U5: renamed from U2; footprint (none) -> Daniel_Kopp:DIP-14_300_ELL
Connections:
- net D0: now also U5.12; no longer U5.4
- net D1: now also U5.1; no longer U5.9
- net Out: now also U3.3; no longer U3.6
- net Select: now also U5.2; no longer U5.10
- net at U2.4: now also U5.13; no longer U5.5
- new net: U3.1, U5.11
- new net: U3.2, U5.3
Changed lines of the file:
@@
 $Descr A4 11693 8268
 encoding utf-8
-Sheet 6 451
+Sheet 6 456
 Title "1:2 Multiplexer"
 Date "2018-09-14"
@@
 Out
 $Comp
-L 4-bit_processor-rescue:74LS32 U3
-U 2 1 5B98DCD8
+L 4-bit_processor-rescue:74LS32 U?
+U 1 1 5B98DCD8
 P 7100 3750
-AR Path="/5B990C59/5B990C5E/5B98DA2C/5B98DCD8" Ref="U3"  Part="2"
-AR Path="/5B990C59/5B99BC00/5B98DA2C/5B98DCD8" Ref="U11"  Part="2"
-AR Path="/5B990C59/5B99C896/5B98DA2C/5B98DCD8" Ref="U19"  Part="2"
-AR Path="/5B990C59/5B99C8B8/5B98DA2C/5B98DCD8" Ref="U26"  Part="2"
-AR Path="/5B9D167A/5B9D1E00/5B990C5E/5B98DA2C/5B98DCD8" Ref="U19"  Part="2"
-AR Path="/5B9D167A/5B9D1E00/5B99BC00/5B98DA2C/5B98DCD8" Ref="U19"  Part="2"
-AR Path="/5B9D167A/5B9D1E00/5B99C896/5B98DA2C/5B98DCD8" Ref="U19"  Part="2"
-AR Path="/5B9D167A/5B9D1E00/5B99C8B8/5B98DA2C/5B98DCD8" Ref="U19"  Part="2"
-F 0 "U19" H 7100 3800 50  0000 C CNN
+AR Path="/5B990C59/5B990C5E/5B98DA2C/5B98DCD8" Ref="U?"  Part="2"
+AR Path="/5B990C59/5B99BC00/5B98DA2C/5B98DCD8" Ref="U?"  Part="2"
+AR Path="/5B990C59/5B99C896/5B98DA2C/5B98DCD8" Ref="U?"  Part="2"
+AR Path="/5B990C59/5B99C8B8/5B98DA2C/5B98DCD8" Ref="U?"  Part="2"
+AR Path="/5B9D167A/5B9D1E00/5B990C5E/5B98DA2C/5B98DCD8" Ref="U3"  Part="2"
+AR Path="/5B9D167A/5B9D1E00/5B99BC00/5B98DA2C/5B98DCD8" Ref="U8"  Part="3"
+AR Path="/5B9D167A/5B9D1E00/5B99C896/5B98DA2C/5B98DCD8" Ref="U13"  Part="4"
+AR Path="/5B9D167A/5B9D1E00/5B99C8B8/5B98DA2C/5B98DCD8" Ref="U22"  Part="1"
+F 0 "U22" H 7100 3800 50  0000 C CNN
 F 1 "74LS32" H 7100 3700 50  0000 C CNN
-F 2 "" H 7100 3750 50  0001 C CNN
+F 2 "Daniel_Kopp:DIP-14_300_ELL" H 7100 3750 50  0001 C CNN
 F 3 "" H 7100 3750 50  0001 C CNN
-	2    7100 3750
+	1    7100 3750
 	1    0    0    -1
 $EndComp
 $Comp
-L 4-bit_processor-rescue:74LS08 U2
-U 2 1 5B98DCDF
+L 4-bit_processor-rescue:74LS08 U?
+U 4 1 5B98DCDF
 P 5750 3350
-AR Path="/5B990C59/5B990C5E/5B98DA2C/5B98DCDF" Ref="U2"  Part="4"
-AR Path="/5B990C59/5B99BC00/5B98DA2C/5B98DCDF" Ref="U13"  Part="1"
-AR Path="/5B990C59/5B99C896/5B98DA2C/5B98DCDF" Ref="U21"  Part="2"
-AR Path="/5B990C59/5B99C8B8/5B98DA2C/5B98DCDF" Ref="U28"  Part="3"
-AR Path="/5B9D167A/5B9D1E00/5B990C5E/5B98DA2C/5B98DCDF" Ref="U21"  Part="2"
-AR Path="/5B9D167A/5B9D1E00/5B99BC00/5B98DA2C/5B98DCDF" Ref="U21"  Part="2"
-AR Path="/5B9D167A/5B9D1E00/5B99C896/5B98DA2C/5B98DCDF" Ref="U21"  Part="2"
-AR Path="/5B9D167A/5B9D1E00/5B99C8B8/5B98DA2C/5B98DCDF" Ref="U21"  Part="2"
-F 0 "U21" H 5750 3400 50  0000 C CNN
+AR Path="/5B990C59/5B990C5E/5B98DA2C/5B98DCDF" Ref="U?"  Part="4"
+AR Path="/5B990C59/5B99BC00/5B98DA2C/5B98DCDF" Ref="U?"  Part="1"
+AR Path="/5B990C59/5B99C896/5B98DA2C/5B98DCDF" Ref="U?"  Part="2"
+AR Path="/5B990C59/5B99C8B8/5B98DA2C/5B98DCDF" Ref="U?"  Part="3"
+AR Path="/5B9D167A/5B9D1E00/5B990C5E/5B98DA2C/5B98DCDF" Ref="U5"  Part="1"
+AR Path="/5B9D167A/5B9D1E00/5B99BC00/5B98DA2C/5B98DCDF" Ref="U10"  Part="2"
+AR Path="/5B9D167A/5B9D1E00/5B99C896/5B98DA2C/5B98DCDF" Ref="U15"  Part="3"
+AR Path="/5B9D167A/5B9D1E00/5B99C8B8/5B98DA2C/5B98DCDF" Ref="U19"  Part="4"
+F 0 "U19" H 5750 3400 50  0000 C CNN
 F 1 "74LS08" H 5750 3300 50  0000 C CNN
-F 2 "" H 5750 3350 50  0001 C CNN
+F 2 "Daniel_Kopp:DIP-14_300_ELL" H 5750 3350 50  0001 C CNN
 F 3 "" H 5750 3350 50  0001 C CNN
-	2    5750 3350
+	4    5750 3350
 	1    0    0    -1
 $EndComp
 $Comp
-L 4-bit_processor-rescue:74LS08 U5
-U 3 1 5B98DCE6
+L 4-bit_processor-rescue:74LS08 U?
+U 1 1 5B98DCE6
 P 5750 4150
-AR Path="/5B990C59/5B990C5E/5B98DA2C/5B98DCE6" Ref="U5"  Part="1"
-AR Path="/5B990C59/5B99BC00/5B98DA2C/5B98DCE6" Ref="U13"  Part="2"
-AR Path="/5B990C59/5B99C896/5B98DA2C/5B98DCE6" Ref="U21"  Part="3"
-AR Path="/5B990C59/5B99C8B8/5B98DA2C/5B98DCE6" Ref="U28"  Part="4"
-AR Path="/5B9D167A/5B9D1E00/5B990C5E/5B98DA2C/5B98DCE6" Ref="U21"  Part="3"
-AR Path="/5B9D167A/5B9D1E00/5B99BC00/5B98DA2C/5B98DCE6" Ref="U21"  Part="3"
-AR Path="/5B9D167A/5B9D1E00/5B99C896/5B98DA2C/5B98DCE6" Ref="U21"  Part="3"
-AR Path="/5B9D167A/5B9D1E00/5B99C8B8/5B98DA2C/5B98DCE6" Ref="U21"  Part="3"
+AR Path="/5B990C59/5B990C5E/5B98DA2C/5B98DCE6" Ref="U?"  Part="1"
+AR Path="/5B990C59/5B99BC00/5B98DA2C/5B98DCE6" Ref="U?"  Part="2"
+AR Path="/5B990C59/5B99C896/5B98DA2C/5B98DCE6" Ref="U?"  Part="3"
+AR Path="/5B990C59/5B99C8B8/5B98DA2C/5B98DCE6" Ref="U?"  Part="4"
+AR Path="/5B9D167A/5B9D1E00/5B990C5E/5B98DA2C/5B98DCE6" Ref="U5"  Part="2"
+AR Path="/5B9D167A/5B9D1E00/5B99BC00/5B98DA2C/5B98DCE6" Ref="U10"  Part="3"
+AR Path="/5B9D167A/5B9D1E00/5B99C896/5B98DA2C/5B98DCE6" Ref="U15"  Part="4"
+AR Path="/5B9D167A/5B9D1E00/5B99C8B8/5B98DA2C/5B98DCE6" Ref="U21"  Part="1"
 F 0 "U21" H 5750 4200 50  0000 C CNN
 F 1 "74LS08" H 5750 4100 50  0000 C CNN
-F 2 "" H 5750 4150 50  0001 C CNN
+F 2 "Daniel_Kopp:DIP-14_300_ELL" H 5750 4150 50  0001 C CNN
 F 3 "" H 5750 4150 50  0001 C CNN
-	3    5750 4150
+	1    5750 4150
 	1    0    0    -1
 $EndComp
@@
 	6500 3350 6350 3350
 $Comp
-L 4-bit_processor-rescue:74LS04 U1
+L 4-bit_processor-rescue:74LS04 U?
 U 2 1 5B98DCF1
 P 4750 2700
-AR Path="/5B990C59/5B990C5E/5B98DA2C/5B98DCF1" Ref="U1"  Part="2"
-AR Path="/5B990C59/5B99BC00/5B98DA2C/5B98DCF1" Ref="U10"  Part="2"
-AR Path="/5B990C59/5B99C896/5B98DA2C/5B98DCF1" Ref="U18"  Part="2"
-AR Path="/5B990C59/5B99C8B8/5B98DA2C/5B98DCF1" Ref="U25"  Part="2"
-AR Path="/5B9D167A/5B9D1E00/5B990C5E/5B98DA2C/5B98DCF1" Ref="U18"  Part="2"
-AR Path="/5B9D167A/5B9D1E00/5B99BC00/5B98DA2C/5B98DCF1" Ref="U18"  Part="2"
-AR Path="/5B9D167A/5B9D1E00/5B99C896/5B98DA2C/5B98DCF1" Ref="U18"  Part="2"
+AR Path="/5B990C59/5B990C5E/5B98DA2C/5B98DCF1" Ref="U?"  Part="2"
+AR Path="/5B990C59/5B99BC00/5B98DA2C/5B98DCF1" Ref="U?"  Part="2"
+AR Path="/5B990C59/5B99C896/5B98DA2C/5B98DCF1" Ref="U?"  Part="2"
+AR Path="/5B990C59/5B99C8B8/5B98DA2C/5B98DCF1" Ref="U?"  Part="2"
+AR Path="/5B9D167A/5B9D1E00/5B990C5E/5B98DA2C/5B98DCF1" Ref="U2"  Part="2"
+AR Path="/5B9D167A/5B9D1E00/5B99BC00/5B98DA2C/5B98DCF1" Ref="U2"  Part="6"
+AR Path="/5B9D167A/5B9D1E00/5B99C896/5B98DA2C/5B98DCF1" Ref="U11"  Part="4"
 AR Path="/5B9D167A/5B9D1E00/5B99C8B8/5B98DA2C/5B98DCF1" Ref="U18"  Part="2"
 F 0 "U18" H 4945 2815 50  0000 C CNN
 F 1 "74LS04" H 4940 2575 50  0000 C CNN
-F 2 "" H 4750 2700 50  0001 C CNN
+F 2 "Daniel_Kopp:DIP-14_300_ELL" H 4750 2700 50  0001 C CNN
 F 3 "" H 4750 2700 50  0001 C CNN
 	2    4750 2700
