File: Potential Schematics/16-1_OR_GATE.sch (KiCad schematic (older format))
At the start: 6 parts, among them U11 74LS32, U17 74LS32, U19 74LS32, U203 74LS32, U204 74LS32, U36 74LS32

Commit message: Adding Multiply Devide
Parts:
- U11, U17, U19, U203, U204, U36: symbol 74LS32 -> 4-bit_processor-rescue:74LS32
Changed lines of the file:
@@
-EESchema Schematic File Version 2
-LIBS:power
-LIBS:device
-LIBS:switches
-LIBS:relays
-LIBS:motors
-LIBS:transistors
-LIBS:conn
-LIBS:linear
-LIBS:regul
-LIBS:74xx
-LIBS:cmos4000
-LIBS:adc-dac
-LIBS:memory
-LIBS:xilinx
-LIBS:microcontrollers
-LIBS:dsp
-LIBS:microchip
-LIBS:analog_switches
-LIBS:motorola
-LIBS:texas
-LIBS:intel
-LIBS:audio
-LIBS:interface
-LIBS:digital-audio
-LIBS:philips
-LIBS:display
-LIBS:cypress
-LIBS:siliconi
-LIBS:opto
-LIBS:atmel
-LIBS:contrib
-LIBS:valves
+EESchema Schematic File Version 4
 LIBS:4-bit_processor-cache
-EELAYER 25 0
+EELAYER 26 0
 EELAYER END
 $Descr A4 11693 8268
 encoding utf-8
-Sheet 423 449
+Sheet 423 451
 Title "16:1 OR"
 Date "2018-09-14"
@@
 Q
 $Comp
-L 74LS32 U11
+L 4-bit_processor-rescue:74LS32 U11
 U 2 1 5BB0EE01
 P 3600 2150
@@
 $EndComp
 $Comp
-L 74LS32 U11
+L 4-bit_processor-rescue:74LS32 U11
 U 3 1 5BB0EE08
 P 4100 2150
@@
 $EndComp
 $Comp
-L 74LS32 U19
+L 4-bit_processor-rescue:74LS32 U19
 U 4 1 5BB0EE0F
 P 4550 2150
@@
 $EndComp
 $Comp
-L 74LS32 U19
+L 4-bit_processor-rescue:74LS32 U19
 U 2 1 5BB0EE16
 P 5050 2150
@@
 $EndComp
 $Comp
-L 74LS32 U36
+L 4-bit_processor-rescue:74LS32 U36
 U 2 1 5BB0EE1D
 P 5500 2150
@@
 $EndComp
 $Comp
-L 74LS32 U203
+L 4-bit_processor-rescue:74LS32 U203
 U 1 1 5BB0EE24
 P 6000 2150
@@
 $EndComp
 $Comp
-L 74LS32 U204
+L 4-bit_processor-rescue:74LS32 U204
 U 3 1 5BB0EE2B
 P 6450 2150
@@
 $EndComp
 $Comp
-L 74LS32 U204
+L 4-bit_processor-rescue:74LS32 U204
 U 4 1 5BB0EE32
 P 6950 2150
@@
 $EndComp
 $Comp
-L 74LS32 U19
+L 4-bit_processor-rescue:74LS32 U19
 U 1 1 5BB0EE39
 P 4550 3750
@@
 $EndComp
 $Comp
-L 74LS32 U17
+L 4-bit_processor-rescue:74LS32 U17
 U 3 1 5BB0EE40
 P 5050 3750
@@
 $EndComp
 $Comp
-L 74LS32 U203
+L 4-bit_processor-rescue:74LS32 U203
 U 3 1 5BB0EE47
 P 5500 3750
@@
 $EndComp
 $Comp
-L 74LS32 U203
+L 4-bit_processor-rescue:74LS32 U203
 U 2 1 5BB0EE4E
 P 6000 3750
@@
 $EndComp
 $Comp
-L 74LS32 U17
+L 4-bit_processor-rescue:74LS32 U17
 U 4 1 5BB0EE55
 P 5050 5100
@@
 $EndComp
 $Comp
-L 74LS32 U203
+L 4-bit_processor-rescue:74LS32 U203
 U 4 1 5BB0EE5C
 P 5550 5100
@@
 $EndComp
 $Comp
-L 74LS32 U36
+L 4-bit_processor-rescue:74LS32 U36
 U 1 1 5BB0EE63
 P 5300 6750

Commit message: Finished PCB
Parts:
- U217: renamed from U19; footprint (none) -> Daniel_Kopp:DIP-14_300_ELL
- U217, U218: renamed from U17; footprint (none) -> Daniel_Kopp:DIP-14_300_ELL
- U218: renamed from U36; footprint (none) -> Daniel_Kopp:DIP-14_300_ELL
- U218, U219: renamed from U203; footprint (none) -> Daniel_Kopp:DIP-14_300_ELL
- U219, U220: renamed from U204; footprint (none) -> Daniel_Kopp:DIP-14_300_ELL
- U27: renamed from U11; footprint (none) -> Daniel_Kopp:DIP-14_300_ELL
Connections:
- net D0: now also U27.13; no longer U27.5
- net D1: now also U27.12; no longer U27.4
- net D2: now also U27.2; no longer U27.10
- net D3: now also U27.1; no longer U27.9
- net D4: now also U217.5; no longer U217.13
- net D5: now also U217.4; no longer U217.12
- net D6: now also U217.13; no longer U217.5
- net D7: now also U217.12; no longer U217.4
- net D8: now also U218.13; no longer U218.5
- net D9: now also U218.12; no longer U218.4
- net Da: now also U219.10; no longer U219.2
- net Db: now also U219.9; no longer U219.1
- net Dc: now also U219.2; no longer U219.10
- net Dd: now also U219.1; no longer U219.9
- net De: now also U220.5; no longer U220.13
- net Df: now also U220.4; no longer U220.12
- net Q: now also U218.8; no longer U218.3
- new net: U217.10, U27.11
- new net: U217.9, U27.3
- new net: U217.2, U217.6
- new net: U217.1, U217.11
- new net: U218.11, U218.2
- new net: U218.1, U219.8
- new net: U219.13, U219.3
- new net: U219.12, U220.6
- new net: U217.8, U218.5
- new net: U217.3, U218.4
- new net: U218.3, U219.5
- new net: U219.11, U219.4
- new net: U218.10, U218.6
- new net: U218.9, U219.6
