File: Potential Schematics/4-bit_Register.sch (KiCad schematic (older format))
At the start: 0 parts

Commit message: Finished PCB
Connections:
- wire segments 25 -> 28
Changed lines of the file:
@@
 $Descr A4 11693 8268
 encoding utf-8
-Sheet 24 451
+Sheet 24 456
 Title "4-bit Register"
 Date "2018-09-14"
@@
 C
 Wire Wire Line
-	1300 5300 5100 5300
+	1300 5300 4250 5300
 Wire Wire Line
-	4250 2450 4250 5300
+	4250 2450 4250 3400
 Wire Wire Line
 	4250 4350 5100 4350
@@
 Wire Wire Line
 	2350 3900 5100 3900
-Wire Wire Line
-	1250 2300 1400 2300
 Wire Wire Line
 	1400 2300 1400 4850
@@
 Wire Wire Line
 	8850 4850 6250 4850
+Wire Wire Line
+	4250 5300 5100 5300
+Wire Wire Line
+	4250 4350 4250 5300
+Wire Wire Line
+	4250 3400 4250 4350
+Wire Wire Line
+	1300 2300 1400 2300
 $EndSCHEMATC
