File: Potential Schematics/4_IN-ANDsch.sch (KiCad schematic (older format))
At the start: 1 part, among them U179 74LS09

Commit message: Adding Multiply Devide
Parts:
- U179: symbol 74LS09 -> 4-bit_processor-rescue:74LS09
Changed lines of the file:
@@
-EESchema Schematic File Version 2
-LIBS:power
-LIBS:device
-LIBS:switches
-LIBS:relays
-LIBS:motors
-LIBS:transistors
-LIBS:conn
-LIBS:linear
-LIBS:regul
-LIBS:74xx
-LIBS:cmos4000
-LIBS:adc-dac
-LIBS:memory
-LIBS:xilinx
-LIBS:microcontrollers
-LIBS:dsp
-LIBS:microchip
-LIBS:analog_switches
-LIBS:motorola
-LIBS:texas
-LIBS:intel
-LIBS:audio
-LIBS:interface
-LIBS:digital-audio
-LIBS:philips
-LIBS:display
-LIBS:cypress
-LIBS:siliconi
-LIBS:opto
-LIBS:atmel
-LIBS:contrib
-LIBS:valves
+EESchema Schematic File Version 4
 LIBS:4-bit_processor-cache
-EELAYER 25 0
+EELAYER 26 0
 EELAYER END
 $Descr A4 11693 8268
 encoding utf-8
-Sheet 361 449
+Sheet 361 451
 Title "Quad In AND"
 Date "2018-09-14"
@@
 Q
 $Comp
-L 74LS09 U179
+L 4-bit_processor-rescue:74LS09 U179
 U 2 1 5B9E5866
 P 3050 2650
@@
 $EndComp
 $Comp
-L 74LS09 U179
+L 4-bit_processor-rescue:74LS09 U179
 U 3 1 5B9E588B
 P 3100 4250
@@
 	2300 4350 2500 4350
 $Comp
-L 74LS09 U179
+L 4-bit_processor-rescue:74LS09 U179
 U 4 1 5B9E59D7
 P 5850 3400

Commit message: Finished PCB
Parts:
- U193: renamed from U179; footprint (none) -> Daniel_Kopp:DIP-14_300_ELL
Changed lines of the file:
@@
 $Descr A4 11693 8268
 encoding utf-8
-Sheet 361 451
+Sheet 364 456
 Title "Quad In AND"
 Date "2018-09-14"
@@
 Q
 $Comp
-L 4-bit_processor-rescue:74LS09 U179
-U 2 1 5B9E5866
+L 4-bit_processor-rescue:74LS09 U193
+U 3 1 5B9E5866
 P 3050 2650
-AR Path="/5B9D167A/5B9C0EA0/5B9E4FB9/5B9E57DB/5B9E5866" Ref="U179"  Part="2"
-AR Path="/5B9D167A/5B9C0EA0/5B9E4FB9/5B9E648A/5B9E5866" Ref="U182"  Part="1"
-AR Path="/5B9D167A/5B9C0EA0/5B9E4FB9/5B9E6A31/5B9E5866" Ref="U182"  Part="4"
-AR Path="/5B9D167A/5B9C0EA0/5B9E4FB9/5B9E6A38/5B9E5866" Ref="U183"  Part="3"
-AR Path="/5B9D167A/5B9C0EA0/5B9E4FB9/5B9E744B/5B9E5866" Ref="U184"  Part="2"
-AR Path="/5B9D167A/5B9C0EA0/5B9E4FB9/5B9E7452/5B9E5866" Ref="U185"  Part="1"
-AR Path="/5B9D167A/5B9C0EA0/5B9E4FB9/5B9E7459/5B9E5866" Ref="U185"  Part="4"
-AR Path="/5B9D167A/5B9C0EA0/5B9E4FB9/5B9E7460/5B9E5866" Ref="U186"  Part="3"
-AR Path="/5B9D167A/5B9C0EA0/5B9E4FB9/5B9E8B97/5B9E5866" Ref="U187"  Part="2"
-AR Path="/5B9D167A/5B9C0EA0/5B9E4FB9/5B9E8B9E/5B9E5866" Ref="U188"  Part="1"
-AR Path="/5B9D167A/5B9C0EA0/5B9E4FB9/5B9E8BA5/5B9E5866" Ref="U188"  Part="4"
-AR Path="/5B9D167A/5B9C0EA0/5B9E4FB9/5B9E8BAC/5B9E5866" Ref="U189"  Part="3"
-AR Path="/5B9D167A/5B9C0EA0/5B9E4FB9/5B9E8BB3/5B9E5866" Ref="U190"  Part="2"
-AR Path="/5B9D167A/5B9C0EA0/5B9E4FB9/5B9E8BBA/5B9E5866" Ref="U191"  Part="1"
-AR Path="/5B9D167A/5B9C0EA0/5B9E4FB9/5B9E8BC1/5B9E5866" Ref="U191"  Part="4"
-AR Path="/5B9D167A/5B9C0EA0/5B9E4FB9/5B9E8BC8/5B9E5866" Ref="U192"  Part="3"
-F 0 "U179" H 3050 2700 50  0000 C CNN
+AR Path="/5B9D167A/5B9C0EA0/5B9E4FB9/5B9E57DB/5B9E5866" Ref="U193"  Part="2"
+AR Path="/5B9D167A/5B9C0EA0/5B9E4FB9/5B9E648A/5B9E5866" Ref="U196"  Part="1"
+AR Path="/5B9D167A/5B9C0EA0/5B9E4FB9/5B9E6A31/5B9E5866" Ref="U196"  Part="4"
+AR Path="/5B9D167A/5B9C0EA0/5B9E4FB9/5B9E6A38/5B9E5866" Ref="U197"  Part="3"
+AR Path="/5B9D167A/5B9C0EA0/5B9E4FB9/5B9E744B/5B9E5866" Ref="U198"  Part="2"
+AR Path="/5B9D167A/5B9C0EA0/5B9E4FB9/5B9E7452/5B9E5866" Ref="U199"  Part="1"
+AR Path="/5B9D167A/5B9C0EA0/5B9E4FB9/5B9E7459/5B9E5866" Ref="U199"  Part="4"
+AR Path="/5B9D167A/5B9C0EA0/5B9E4FB9/5B9E7460/5B9E5866" Ref="U200"  Part="3"
+AR Path="/5B9D167A/5B9C0EA0/5B9E4FB9/5B9E8B97/5B9E5866" Ref="U201"  Part="2"
+AR Path="/5B9D167A/5B9C0EA0/5B9E4FB9/5B9E8B9E/5B9E5866" Ref="U202"  Part="1"
+AR Path="/5B9D167A/5B9C0EA0/5B9E4FB9/5B9E8BA5/5B9E5866" Ref="U202"  Part="4"
+AR Path="/5B9D167A/5B9C0EA0/5B9E4FB9/5B9E8BAC/5B9E5866" Ref="U203"  Part="3"
+AR Path="/5B9D167A/5B9C0EA0/5B9E4FB9/5B9E8BB3/5B9E5866" Ref="U204"  Part="2"
+AR Path="/5B9D167A/5B9C0EA0/5B9E4FB9/5B9E8BBA/5B9E5866" Ref="U205"  Part="1"
+AR Path="/5B9D167A/5B9C0EA0/5B9E4FB9/5B9E8BC1/5B9E5866" Ref="U205"  Part="4"
+AR Path="/5B9D167A/5B9C0EA0/5B9E4FB9/5B9E8BC8/5B9E5866" Ref="U206"  Part="3"
+F 0 "U206" H 3050 2700 50  0000 C CNN
 F 1 "74LS09" H 3050 2600 50  0000 C CNN
-F 2 "" H 3050 2650 50  0001 C CNN
+F 2 "Daniel_Kopp:DIP-14_300_ELL" H 3050 2650 50  0001 C CNN
 F 3 "" H 3050 2650 50  0001 C CNN
-	2    3050 2650
+	3    3050 2650
 	1    0    0    -1
 $EndComp
 $Comp
-L 4-bit_processor-rescue:74LS09 U179
-U 3 1 5B9E588B
+L 4-bit_processor-rescue:74LS09 U193
+U 4 1 5B9E588B
 P 3100 4250
-AR Path="/5B9D167A/5B9C0EA0/5B9E4FB9/5B9E57DB/5B9E588B" Ref="U179"  Part="3"
-AR Path="/5B9D167A/5B9C0EA0/5B9E4FB9/5B9E648A/5B9E588B" Ref="U182"  Part="2"
-AR Path="/5B9D167A/5B9C0EA0/5B9E4FB9/5B9E6A31/5B9E588B" Ref="U183"  Part="1"
-AR Path="/5B9D167A/5B9C0EA0/5B9E4FB9/5B9E6A38/5B9E588B" Ref="U183"  Part="4"
-AR Path="/5B9D167A/5B9C0EA0/5B9E4FB9/5B9E744B/5B9E588B" Ref="U184"  Part="3"
-AR Path="/5B9D167A/5B9C0EA0/5B9E4FB9/5B9E7452/5B9E588B" Ref="U185"  Part="2"
-AR Path="/5B9D167A/5B9C0EA0/5B9E4FB9/5B9E7459/5B9E588B" Ref="U186"  Part="1"
-AR Path="/5B9D167A/5B9C0EA0/5B9E4FB9/5B9E7460/5B9E588B" Ref="U186"  Part="4"
-AR Path="/5B9D167A/5B9C0EA0/5B9E4FB9/5B9E8B97/5B9E588B" Ref="U187"  Part="3"
-AR Path="/5B9D167A/5B9C0EA0/5B9E4FB9/5B9E8B9E/5B9E588B" Ref="U188"  Part="2"
-AR Path="/5B9D167A/5B9C0EA0/5B9E4FB9/5B9E8BA5/5B9E588B" Ref="U189"  Part="1"
-AR Path="/5B9D167A/5B9C0EA0/5B9E4FB9/5B9E8BAC/5B9E588B" Ref="U189"  Part="4"
-AR Path="/5B9D167A/5B9C0EA0/5B9E4FB9/5B9E8BB3/5B9E588B" Ref="U190"  Part="3"
-AR Path="/5B9D167A/5B9C0EA0/5B9E4FB9/5B9E8BBA/5B9E588B" Ref="U191"  Part="2"
-AR Path="/5B9D167A/5B9C0EA0/5B9E4FB9/5B9E8BC1/5B9E588B" Ref="U192"  Part="1"
-AR Path="/5B9D167A/5B9C0EA0/5B9E4FB9/5B9E8BC8/5B9E588B" Ref="U192"  Part="4"
-F 0 "U179" H 3100 4300 50  0000 C CNN
+AR Path="/5B9D167A/5B9C0EA0/5B9E4FB9/5B9E57DB/5B9E588B" Ref="U193"  Part="3"
+AR Path="/5B9D167A/5B9C0EA0/5B9E4FB9/5B9E648A/5B9E588B" Ref="U196"  Part="2"
+AR Path="/5B9D167A/5B9C0EA0/5B9E4FB9/5B9E6A31/5B9E588B" Ref="U197"  Part="1"
+AR Path="/5B9D167A/5B9C0EA0/5B9E4FB9/5B9E6A38/5B9E588B" Ref="U197"  Part="4"
+AR Path="/5B9D167A/5B9C0EA0/5B9E4FB9/5B9E744B/5B9E588B" Ref="U198"  Part="3"
+AR Path="/5B9D167A/5B9C0EA0/5B9E4FB9/5B9E7452/5B9E588B" Ref="U199"  Part="2"
+AR Path="/5B9D167A/5B9C0EA0/5B9E4FB9/5B9E7459/5B9E588B" Ref="U200"  Part="1"
+AR Path="/5B9D167A/5B9C0EA0/5B9E4FB9/5B9E7460/5B9E588B" Ref="U200"  Part="4"
+AR Path="/5B9D167A/5B9C0EA0/5B9E4FB9/5B9E8B97/5B9E588B" Ref="U201"  Part="3"
+AR Path="/5B9D167A/5B9C0EA0/5B9E4FB9/5B9E8B9E/5B9E588B" Ref="U202"  Part="2"
+AR Path="/5B9D167A/5B9C0EA0/5B9E4FB9/5B9E8BA5/5B9E588B" Ref="U203"  Part="1"
+AR Path="/5B9D167A/5B9C0EA0/5B9E4FB9/5B9E8BAC/5B9E588B" Ref="U203"  Part="4"
+AR Path="/5B9D167A/5B9C0EA0/5B9E4FB9/5B9E8BB3/5B9E588B" Ref="U204"  Part="3"
+AR Path="/5B9D167A/5B9C0EA0/5B9E4FB9/5B9E8BBA/5B9E588B" Ref="U205"  Part="2"
+AR Path="/5B9D167A/5B9C0EA0/5B9E4FB9/5B9E8BC1/5B9E588B" Ref="U206"  Part="1"
+AR Path="/5B9D167A/5B9C0EA0/5B9E4FB9/5B9E8BC8/5B9E588B" Ref="U206"  Part="4"
+F 0 "U206" H 3100 4300 50  0000 C CNN
 F 1 "74LS09" H 3100 4200 50  0000 C CNN
-F 2 "" H 3100 4250 50  0001 C CNN
+F 2 "Daniel_Kopp:DIP-14_300_ELL" H 3100 4250 50  0001 C CNN
 F 3 "" H 3100 4250 50  0001 C CNN
-	3    3100 4250
+	4    3100 4250
 	1    0    0    -1
 $EndComp
@@
 	2300 4350 2500 4350
 $Comp
-L 4-bit_processor-rescue:74LS09 U179
-U 4 1 5B9E59D7
+L 4-bit_processor-rescue:74LS09 U193
+U 1 1 5B9E59D7
 P 5850 3400
-AR Path="/5B9D167A/5B9C0EA0/5B9E4FB9/5B9E57DB/5B9E59D7" Ref="U179"  Part="4"
-AR Path="/5B9D167A/5B9C0EA0/5B9E4FB9/5B9E648A/5B9E59D7" Ref="U182"  Part="3"
-AR Path="/5B9D167A/5B9C0EA0/5B9E4FB9/5B9E6A31/5B9E59D7" Ref="U183"  Part="2"
-AR Path="/5B9D167A/5B9C0EA0/5B9E4FB9/5B9E6A38/5B9E59D7" Ref="U184"  Part="1"
-AR Path="/5B9D167A/5B9C0EA0/5B9E4FB9/5B9E744B/5B9E59D7" Ref="U184"  Part="4"
-AR Path="/5B9D167A/5B9C0EA0/5B9E4FB9/5B9E7452/5B9E59D7" Ref="U185"  Part="3"
-AR Path="/5B9D167A/5B9C0EA0/5B9E4FB9/5B9E7459/5B9E59D7" Ref="U186"  Part="2"
-AR Path="/5B9D167A/5B9C0EA0/5B9E4FB9/5B9E7460/5B9E59D7" Ref="U187"  Part="1"
-AR Path="/5B9D167A/5B9C0EA0/5B9E4FB9/5B9E8B97/5B9E59D7" Ref="U187"  Part="4"
-AR Path="/5B9D167A/5B9C0EA0/5B9E4FB9/5B9E8B9E/5B9E59D7" Ref="U188"  Part="3"
-AR Path="/5B9D167A/5B9C0EA0/5B9E4FB9/5B9E8BA5/5B9E59D7" Ref="U189"  Part="2"
-AR Path="/5B9D167A/5B9C0EA0/5B9E4FB9/5B9E8BAC/5B9E59D7" Ref="U190"  Part="1"
-AR Path="/5B9D167A/5B9C0EA0/5B9E4FB9/5B9E8BB3/5B9E59D7" Ref="U190"  Part="4"
-AR Path="/5B9D167A/5B9C0EA0/5B9E4FB9/5B9E8BBA/5B9E59D7" Ref="U191"  Part="3"
-AR Path="/5B9D167A/5B9C0EA0/5B9E4FB9/5B9E8BC1/5B9E59D7" Ref="U192"  Part="2"
-AR Path="/5B9D167A/5B9C0EA0/5B9E4FB9/5B9E8BC8/5B9E59D7" Ref="U193"  Part="1"
-F 0 "U179" H 5850 3450 50  0000 C CNN
+AR Path="/5B9D167A/5B9C0EA0/5B9E4FB9/5B9E57DB/5B9E59D7" Ref="U193"  Part="4"
+AR Path="/5B9D167A/5B9C0EA0/5B9E4FB9/5B9E648A/5B9E59D7" Ref="U196"  Part="3"
+AR Path="/5B9D167A/5B9C0EA0/5B9E4FB9/5B9E6A31/5B9E59D7" Ref="U197"  Part="2"
+AR Path="/5B9D167A/5B9C0EA0/5B9E4FB9/5B9E6A38/5B9E59D7" Ref="U198"  Part="1"
+AR Path="/5B9D167A/5B9C0EA0/5B9E4FB9/5B9E744B/5B9E59D7" Ref="U198"  Part="4"
+AR Path="/5B9D167A/5B9C0EA0/5B9E4FB9/5B9E7452/5B9E59D7" Ref="U199"  Part="3"
+AR Path="/5B9D167A/5B9C0EA0/5B9E4FB9/5B9E7459/5B9E59D7" Ref="U200"  Part="2"
+AR Path="/5B9D167A/5B9C0EA0/5B9E4FB9/5B9E7460/5B9E59D7" Ref="U201"  Part="1"
+AR Path="/5B9D167A/5B9C0EA0/5B9E4FB9/5B9E8B97/5B9E59D7" Ref="U201"  Part="4"
+AR Path="/5B9D167A/5B9C0EA0/5B9E4FB9/5B9E8B9E/5B9E59D7" Ref="U202"  Part="3"
+AR Path="/5B9D167A/5B9C0EA0/5B9E4FB9/5B9E8BA5/5B9E59D7" Ref="U203"  Part="2"
+AR Path="/5B9D167A/5B9C0EA0/5B9E4FB9/5B9E8BAC/5B9E59D7" Ref="U204"  Part="1"
+AR Path="/5B9D167A/5B9C0EA0/5B9E4FB9/5B9E8BB3/5B9E59D7" Ref="U204"  Part="4"
+AR Path="/5B9D167A/5B9C0EA0/5B9E4FB9/5B9E8BBA/5B9E59D7" Ref="U205"  Part="3"
+AR Path="/5B9D167A/5B9C0EA0/5B9E4FB9/5B9E8BC1/5B9E59D7" Ref="U206"  Part="2"
+AR Path="/5B9D167A/5B9C0EA0/5B9E4FB9/5B9E8BC8/5B9E59D7" Ref="U207"  Part="1"
+F 0 "U207" H 5850 3450 50  0000 C CNN
 F 1 "74LS09" H 5850 3350 50  0000 C CNN
-F 2 "" H 5850 3400 50  0001 C CNN
+F 2 "Daniel_Kopp:DIP-14_300_ELL" H 5850 3400 50  0001 C CNN
 F 3 "" H 5850 3400 50  0001 C CNN
-	4    5850 3400
+	1    5850 3400
 	1    0    0    -1
 $EndComp
