File: Potential Schematics/Registers.sch (KiCad schematic (older format))
At the start: 6 parts, among them U18 74LS04, U2 74LS09, U3 74LS09, U4 74LS09, U6 74LS09, U7 74LS09

Commit message: Adding Multiply Devide
Parts:
- U18: symbol 74LS04 -> 4-bit_processor-rescue:74LS04
- U2, U3, U4, U6, U7: symbol 74LS09 -> 4-bit_processor-rescue:74LS09
Changed lines of the file:
@@
-EESchema Schematic File Version 2
-LIBS:power
-LIBS:device
-LIBS:switches
-LIBS:relays
-LIBS:motors
-LIBS:transistors
-LIBS:conn
-LIBS:linear
-LIBS:regul
-LIBS:74xx
-LIBS:cmos4000
-LIBS:adc-dac
-LIBS:memory
-LIBS:xilinx
-LIBS:microcontrollers
-LIBS:dsp
-LIBS:microchip
-LIBS:analog_switches
-LIBS:motorola
-LIBS:texas
-LIBS:intel
-LIBS:audio
-LIBS:interface
-LIBS:digital-audio
-LIBS:philips
-LIBS:display
-LIBS:cypress
-LIBS:siliconi
-LIBS:opto
-LIBS:atmel
-LIBS:contrib
-LIBS:valves
+EESchema Schematic File Version 4
 LIBS:4-bit_processor-cache
-EELAYER 25 0
+EELAYER 26 0
 EELAYER END
 $Descr A4 11693 8268
 encoding utf-8
-Sheet 23 449
+Sheet 23 451
 Title "Registers / Cache"
 Date "2018-09-14"
@@
 Off
 $Comp
-L 74LS09 U2
+L 4-bit_processor-rescue:74LS09 U2
 U 4 1 5B9C957B
 P 3350 7300
@@
 $EndComp
 $Comp
-L 74LS04 U18
+L 4-bit_processor-rescue:74LS04 U18
 U 1 1 5B9CA481
 P 2450 6900
@@
 $EndSheet
 $Comp
-L 74LS09 U2
+L 4-bit_processor-rescue:74LS09 U2
 U 1 1 5BAB5A82
 P 2150 5300
@@
 $EndComp
 $Comp
-L 74LS09 U2
+L 4-bit_processor-rescue:74LS09 U2
 U 2 1 5BAB5B67
 P 2650 5300
@@
 $EndComp
 $Comp
-L 74LS09 U2
+L 4-bit_processor-rescue:74LS09 U2
 U 3 1 5BAB5C8C
 P 3150 5300
@@
 $EndComp
 $Comp
-L 74LS09 U3
+L 4-bit_processor-rescue:74LS09 U3
 U 1 1 5BAB5C92
 P 3650 5300
@@
 $EndComp
 $Comp
-L 74LS09 U3
+L 4-bit_processor-rescue:74LS09 U3
 U 2 1 5BAB5D71
 P 4150 5300
@@
 $EndComp
 $Comp
-L 74LS09 U3
+L 4-bit_processor-rescue:74LS09 U3
 U 3 1 5BAB5D77
 P 4650 5300
@@
 $EndComp
 $Comp
-L 74LS09 U3
+L 4-bit_processor-rescue:74LS09 U3
 U 4 1 5BAB5D7D
 P 5150 5300
@@
 $EndComp
 $Comp
-L 74LS09 U4
+L 4-bit_processor-rescue:74LS09 U4
 U 1 1 5BAB5D83
 P 5650 5300
@@
 $EndComp
 $Comp
-L 74LS09 U4
+L 4-bit_processor-rescue:74LS09 U4
 U 2 1 5BAB5EB6
 P 6150 5300
@@
 $EndComp
 $Comp
-L 74LS09 U4
+L 4-bit_processor-rescue:74LS09 U4
 U 3 1 5BAB5EBC
 P 6650 5300
@@
 $EndComp
 $Comp
-L 74LS09 U4
+L 4-bit_processor-rescue:74LS09 U4
 U 4 1 5BAB5EC2
 P 7150 5300
@@
 $EndComp
 $Comp
-L 74LS09 U6
+L 4-bit_processor-rescue:74LS09 U6
 U 1 1 5BAB5EC8
 P 7650 5300
@@
 $EndComp
 $Comp
-L 74LS09 U6
+L 4-bit_processor-rescue:74LS09 U6
 U 2 1 5BAB5ECE
 P 8150 5300
@@
 $EndComp
 $Comp
-L 74LS09 U6
+L 4-bit_processor-rescue:74LS09 U6
 U 3 1 5BAB5ED4
 P 8650 5300
@@
 $EndComp
 $Comp
-L 74LS09 U6
+L 4-bit_processor-rescue:74LS09 U6
 U 4 1 5BAB5EDA
 P 9150 5300
@@
 $EndComp
 $Comp
-L 74LS09 U7
+L 4-bit_processor-rescue:74LS09 U7
 U 1 1 5BAB5EE0
 P 9650 5300

Commit message: Finished PCB
Parts:
- U25: renamed from U18; footprint (none) -> Daniel_Kopp:DIP-14_300_ELL
- U30: renamed from U2; footprint (none) -> Daniel_Kopp:DIP-14_300_ELL
- U31: renamed from U3; footprint (none) -> Daniel_Kopp:DIP-14_300_ELL
- U32: renamed from U4; footprint (none) -> Daniel_Kopp:DIP-14_300_ELL
- U33: renamed from U6; footprint (none) -> Daniel_Kopp:DIP-14_300_ELL
- U34: renamed from U7; footprint (none) -> Daniel_Kopp:DIP-14_300_ELL
Connections:
- wire segments 364 -> 439
