File: Potential Schematics/selector.sch (KiCad schematic (older format))
At the start: 4 parts, among them U33 74LS04, U34 74LS08, U35 74LS08, U36 74LS32

Commit message: Adding Multiply Devide
Parts:
- U33: symbol 74LS04 -> 4-bit_processor-rescue:74LS04
- U34, U35: symbol 74LS08 -> 4-bit_processor-rescue:74LS08
- U36: symbol 74LS32 -> 4-bit_processor-rescue:74LS32
Changed lines of the file:
@@
-EESchema Schematic File Version 2
-LIBS:power
-LIBS:device
-LIBS:switches
-LIBS:relays
-LIBS:motors
-LIBS:transistors
-LIBS:conn
-LIBS:linear
-LIBS:regul
-LIBS:74xx
-LIBS:cmos4000
-LIBS:adc-dac
-LIBS:memory
-LIBS:xilinx
-LIBS:microcontrollers
-LIBS:dsp
-LIBS:microchip
-LIBS:analog_switches
-LIBS:motorola
-LIBS:texas
-LIBS:intel
-LIBS:audio
-LIBS:interface
-LIBS:digital-audio
-LIBS:philips
-LIBS:display
-LIBS:cypress
-LIBS:siliconi
-LIBS:opto
-LIBS:atmel
-LIBS:contrib
-LIBS:valves
+EESchema Schematic File Version 4
 LIBS:4-bit_processor-cache
-EELAYER 25 0
+EELAYER 26 0
 EELAYER END
 $Descr A4 11693 8268
 encoding utf-8
-Sheet 19 449
+Sheet 19 451
 Title "Decoder/Multiplexer/Selector"
 Date "2018-09-14"
@@
 S2
 $Comp
-L 74LS08 U35
+L 4-bit_processor-rescue:74LS08 U35
 U 1 1 5B9AC09A
 P 7300 4050
@@
 $EndComp
 $Comp
-L 74LS04 U33
+L 4-bit_processor-rescue:74LS04 U33
 U 2 1 5B9AC30F
 P 3850 4400
@@
 Connection ~ 4300 4400
 $Comp
-L 74LS08 U34
+L 4-bit_processor-rescue:74LS08 U34
 U 3 1 5B9ACE5C
 P 7200 2050
@@
 $EndComp
 $Comp
-L 74LS08 U34
+L 4-bit_processor-rescue:74LS08 U34
 U 4 1 5B9ACF0E
 P 7200 2550
@@
 	4500 1950 6600 1950
 $Comp
-L 74LS32 U36
+L 4-bit_processor-rescue:74LS32 U36
 U 1 1 5B9AD025
 P 8650 2150
@@
 $EndComp
 $Comp
-L 74LS32 U36
+L 4-bit_processor-rescue:74LS32 U36
 U 2 1 5B9AD134
 P 8650 2650
@@
 	9350 2250 10100 2250
 $Comp
-L 74LS04 U33
+L 4-bit_processor-rescue:74LS04 U33
 U 1 1 5B9B8AF0
 P 3600 3250
@@
 $EndComp
 $Comp
-L 74LS04 U33
+L 4-bit_processor-rescue:74LS04 U33
 U 3 1 5B9B8C05
 P 4000 3350
@@
 	7900 3000 9250 3000
 $Comp
-L 74LS08 U34
+L 4-bit_processor-rescue:74LS08 U34
 U 1 1 5B9B90AC
 P 4950 3900
@@
 $EndComp
 $Comp
-L 74LS08 U34
+L 4-bit_processor-rescue:74LS08 U34
 U 2 1 5B9B9141
 P 5000 4950

Commit message: Finished PCB
Parts:
- U18, U25: renamed from U33; footprint (none) -> Daniel_Kopp:DIP-14_300_ELL
- U21, U26: renamed from U34; footprint (none) -> Daniel_Kopp:DIP-14_300_ELL
- U26: renamed from U35; footprint (none) -> Daniel_Kopp:DIP-14_300_ELL
- U27: renamed from U36; footprint (none) -> Daniel_Kopp:DIP-14_300_ELL
Connections:
- net OP0: now also U18.11, U21.12; no longer U18.1, U21.9
- net OP1: now also U25.1, U26.1; no longer U25.5, U26.12
- net OP2: now also U21.10; no longer U21.5
- net OP3: now also U18.13; no longer U18.3
- net S2: now also U26.6; no longer U26.3
- net at U27.1: now also U21.11; no longer U21.8
- net at U27.4: now also U26.3; no longer U26.11
- new net: U21.6, U26.4
- new net: U21.8, U26.5
- new net: U18.12, U21.13, U21.9, U26.2
- new net: U18.10, U21.5
- new net: U21.4, U25.2
Changed lines of the file:
@@
 $Descr A4 11693 8268
 encoding utf-8
-Sheet 19 451
+Sheet 19 456
 Title "Decoder/Multiplexer/Selector"
 Date "2018-09-14"
@@
 S2
 $Comp
-L 4-bit_processor-rescue:74LS08 U35
-U 1 1 5B9AC09A
+L 4-bit_processor-rescue:74LS08 U26
+U 2 1 5B9AC09A
 P 7300 4050
-F 0 "U35" H 7300 4100 50  0000 C CNN
+F 0 "U26" H 7300 4100 50  0000 C CNN
 F 1 "74LS08" H 7300 4000 50  0000 C CNN
-F 2 "" H 7300 4050 50  0001 C CNN
+F 2 "Daniel_Kopp:DIP-14_300_ELL" H 7300 4050 50  0001 C CNN
 F 3 "" H 7300 4050 50  0001 C CNN
-	1    7300 4050
+	2    7300 4050
 	1    0    0    -1
 $EndComp
 $Comp
-L 4-bit_processor-rescue:74LS04 U33
-U 2 1 5B9AC30F
+L 4-bit_processor-rescue:74LS04 U18
+U 6 1 5B9AC30F
 P 3850 4400
-F 0 "U33" H 4045 4515 50  0000 C CNN
+F 0 "U18" H 4045 4515 50  0000 C CNN
 F 1 "74LS04" H 4040 4275 50  0000 C CNN
-F 2 "" H 3850 4400 50  0001 C CNN
+F 2 "Daniel_Kopp:DIP-14_300_ELL" H 3850 4400 50  0001 C CNN
 F 3 "" H 3850 4400 50  0001 C CNN
-	2    3850 4400
+	6    3850 4400
 	1    0    0    -1
 $EndComp
@@
 Connection ~ 4300 4400
 $Comp
-L 4-bit_processor-rescue:74LS08 U34
-U 3 1 5B9ACE5C
+L 4-bit_processor-rescue:74LS08 U21
+U 4 1 5B9ACE5C
 P 7200 2050
-F 0 "U34" H 7200 2100 50  0000 C CNN
+F 0 "U21" H 7200 2100 50  0000 C CNN
 F 1 "74LS08" H 7200 2000 50  0000 C CNN
-F 2 "" H 7200 2050 50  0001 C CNN
+F 2 "Daniel_Kopp:DIP-14_300_ELL" H 7200 2050 50  0001 C CNN
 F 3 "" H 7200 2050 50  0001 C CNN
-	3    7200 2050
+	4    7200 2050
 	1    0    0    -1
 $EndComp
 $Comp
-L 4-bit_processor-rescue:74LS08 U34
-U 4 1 5B9ACF0E
+L 4-bit_processor-rescue:74LS08 U26
+U 1 1 5B9ACF0E
 P 7200 2550
-F 0 "U34" H 7200 2600 50  0000 C CNN
+F 0 "U26" H 7200 2600 50  0000 C CNN
 F 1 "74LS08" H 7200 2500 50  0000 C CNN
-F 2 "" H 7200 2550 50  0001 C CNN
+F 2 "Daniel_Kopp:DIP-14_300_ELL" H 7200 2550 50  0001 C CNN
 F 3 "" H 7200 2550 50  0001 C CNN
-	4    7200 2550
+	1    7200 2550
 	1    0    0    -1
 $EndComp
@@
 	4500 1950 6600 1950
 $Comp
-L 4-bit_processor-rescue:74LS32 U36
+L 4-bit_processor-rescue:74LS32 U27
 U 1 1 5B9AD025
 P 8650 2150
-F 0 "U36" H 8650 2200 50  0000 C CNN
+F 0 "U27" H 8650 2200 50  0000 C CNN
 F 1 "74LS32" H 8650 2100 50  0000 C CNN
-F 2 "" H 8650 2150 50  0001 C CNN
+F 2 "Daniel_Kopp:DIP-14_300_ELL" H 8650 2150 50  0001 C CNN
 F 3 "" H 8650 2150 50  0001 C CNN
 	1    8650 2150
@@
 $EndComp
 $Comp
-L 4-bit_processor-rescue:74LS32 U36
+L 4-bit_processor-rescue:74LS32 U27
 U 2 1 5B9AD134
 P 8650 2650
-F 0 "U36" H 8650 2700 50  0000 C CNN
+F 0 "U27" H 8650 2700 50  0000 C CNN
 F 1 "74LS32" H 8650 2600 50  0000 C CNN
-F 2 "" H 8650 2650 50  0001 C CNN
+F 2 "Daniel_Kopp:DIP-14_300_ELL" H 8650 2650 50  0001 C CNN
 F 3 "" H 8650 2650 50  0001 C CNN
 	2    8650 2650
@@
 	9350 2250 10100 2250
 $Comp
-L 4-bit_processor-rescue:74LS04 U33
-U 1 1 5B9B8AF0
+L 4-bit_processor-rescue:74LS04 U18
+U 5 1 5B9B8AF0
 P 3600 3250
-F 0 "U33" H 3795 3365 50  0000 C CNN
+F 0 "U18" H 3795 3365 50  0000 C CNN
 F 1 "74LS04" H 3790 3125 50  0000 C CNN
-F 2 "" H 3600 3250 50  0001 C CNN
+F 2 "Daniel_Kopp:DIP-14_300_ELL" H 3600 3250 50  0001 C CNN
 F 3 "" H 3600 3250 50  0001 C CNN
-	1    3600 3250
+	5    3600 3250
 	0    1    1    0
 $EndComp
 $Comp
-L 4-bit_processor-rescue:74LS04 U33
-U 3 1 5B9B8C05
+L 4-bit_processor-rescue:74LS04 U25
+U 1 1 5B9B8C05
 P 4000 3350
-F 0 "U33" H 4195 3465 50  0000 C CNN
+F 0 "U25" H 4195 3465 50  0000 C CNN
 F 1 "74LS04" H 4190 3225 50  0000 C CNN
-F 2 "" H 4000 3350 50  0001 C CNN
+F 2 "Daniel_Kopp:DIP-14_300_ELL" H 4000 3350 50  0001 C CNN
 F 3 "" H 4000 3350 50  0001 C CNN
-	3    4000 3350
+	1    4000 3350
 	0    1    1    0
 $EndComp
@@
 	7900 3000 9250 3000
 $Comp
-L 4-bit_processor-rescue:74LS08 U34
-U 1 1 5B9B90AC
+L 4-bit_processor-rescue:74LS08 U21
+U 2 1 5B9B90AC
 P 4950 3900
-F 0 "U34" H 4950 3950 50  0000 C CNN
+F 0 "U21" H 4950 3950 50  0000 C CNN
 F 1 "74LS08" H 4950 3850 50  0000 C CNN
-F 2 "" H 4950 3900 50  0001 C CNN
+F 2 "Daniel_Kopp:DIP-14_300_ELL" H 4950 3900 50  0001 C CNN
 F 3 "" H 4950 3900 50  0001 C CNN
-	1    4950 3900
+	2    4950 3900
 	1    0    0    -1
 $EndComp
 $Comp
-L 4-bit_processor-rescue:74LS08 U34
-U 2 1 5B9B9141
+L 4-bit_processor-rescue:74LS08 U21
+U 3 1 5B9B9141
 P 5000 4950
-F 0 "U34" H 5000 5000 50  0000 C CNN
+F 0 "U21" H 5000 5000 50  0000 C CNN
 F 1 "74LS08" H 5000 4900 50  0000 C CNN
-F 2 "" H 5000 4950 50  0001 C CNN
+F 2 "Daniel_Kopp:DIP-14_300_ELL" H 5000 4950 50  0001 C CNN
 F 3 "" H 5000 4950 50  0001 C CNN
-	2    5000 4950
+	3    5000 4950
 	1    0    0    -1
 $EndComp
